Commit message: small update puntilt_description

File: DynamixelPunTilt/puntilt_description/urdf/puntilt_dynamixel-2XL430_realsense-D435.urdf.xacro (robot description, xacro)
@@ -12,5 +12,5 @@
         <parent link="world"/>
         <child link="base"/>
-        <origin xyz="0 0 0.005" rpy="0 0 0"/>
+        <origin xyz="0 0 0" rpy="0 0 0"/>
     </joint>
 	<link name="base" />

Commit message: update

File: DynamixelPunTilt/puntilt_description/urdf/puntilt_dynamixel-2XL430_realsense-D435.urdf.xacro (robot description, xacro)
@@ -8,17 +8,33 @@
     <xacro:arg name="add_plug" default="false" />
     <xacro:arg name="use_mesh" default="true" />
-	<link name="world"/>
-    <joint name="joint_world_base" type="fixed">
-        <parent link="world"/>
-        <child link="base"/>
-        <origin xyz="0 0 0" rpy="0 0 0"/>
+	<link name="base">
+        <visual>
+			<origin xyz="0 0 0" rpy="0 0 0"/>
+			<geometry>
+                <mesh filename="package://puntilt_description/meshes/waffle_base.stl" scale="0.001 0.001 0.001"/>
+			</geometry>
+			<material name="orange"/>
+		</visual>
+        <collision>
+            <origin xyz="0 0 0.047" rpy="0 0 0"/>
+            <geometry>
+                <box size="0.266 0.266 0.094"/>
+            </geometry>
+        </collision>
+        <inertial>
+            <origin xyz="${0} ${0} ${0}" rpy="${0} 0 0"/>
+            <mass value="1000"/>
+            <inertia ixx="1000"  ixy="0.00" ixz="0.00"
+                                 iyy="1000" iyz="0.00"
+                                            izz="1000" />
+        </inertial>
+    </link>
+    <joint name="weld" type="fixed">
+        <parent link="base"/>
+        <child link="puntilt_base"/>
+        <origin xyz="0 0 0.094" rpy="0 0 0"/>
     </joint>
-	<link name="base" />
-    <joint name="joint_base_yaw" type="fixed">
-        <parent link="base"/>
-        <child link="yaw"/>
-    </joint>
-	<link name="yaw">
-        <visual>
+	<link name="puntilt_base">
+        <!-- <visual>
 			<origin xyz="0 0 0" rpy="0 0 0"/>
 			<geometry>
@@ -26,9 +42,9 @@
 			</geometry>
 			<material name="orange"/>
-		</visual>
+		</visual> -->
     </link>
-	<xacro:servo_2XL430 parent="yaw" center_parent="false" child="pitch" center_child="true" />
+	<xacro:servo_2XL430 name_parent="yaw" parent="puntilt_base" center_parent="false" child="pitch" center_child="true" />
 	<link name="pitch">
-		<visual>
+		<!-- <visual>
 			<origin xyz="0 0 0" rpy="0 0 0"/>
 			<geometry>
@@ -36,5 +52,5 @@
 			</geometry>
 			<material name="red"/>
-		</visual>
+		</visual> -->
 	</link>
     <xacro:sensor_d435 parent="pitch" use_nominal_extrinsics="$(arg use_nominal_extrinsics)" add_plug="$(arg add_plug)" use_mesh="$(arg use_mesh)">

File: DynamixelPunTilt/puntilt_description/urdf/puntilt_dynamixel-XM430-double_realsense-D435.urdf.xacro (robot description, xacro)
@@ -8,12 +8,33 @@
     <xacro:arg name="add_plug" default="false" />
     <xacro:arg name="use_mesh" default="true" />
-	<link name="world"/>
-    <joint name="fixed_joint" type="fixed">
-        <parent link="world"/>
-        <child link="base"/>
-        <origin xyz="0 0 0" rpy="0 0 0"/>
+    <link name="base">
+        <visual>
+			<origin xyz="0 0 0" rpy="0 0 0"/>
+			<geometry>
+                <mesh filename="package://puntilt_description/meshes/waffle_base.stl" scale="0.001 0.001 0.001"/>
+			</geometry>
+			<material name="orange"/>
+		</visual>
+        <collision>
+            <origin xyz="0 0 0.047" rpy="0 0 0"/>
+            <geometry>
+                <box size="0.266 0.266 0.094"/>
+            </geometry>
+        </collision>
+        <inertial>
+            <origin xyz="${0} ${0} ${0}" rpy="${0} 0 0"/>
+            <mass value="1000"/>
+            <inertia ixx="1000"  ixy="0.00" ixz="0.00"
+                                 iyy="1000" iyz="0.00"
+                                            izz="1000" />
+        </inertial>
+    </link>
+    <joint name="weld" type="fixed">
+        <parent link="base"/>
+        <child link="puntilt_base"/>
+        <origin xyz="0 0 0.094" rpy="0 0 0"/>
     </joint>
-	<link name="base">
-		<visual>
+	<link name="puntilt_base">
+        <!-- <visual>
 			<origin xyz="0 0 0" rpy="0 0 0"/>
 			<geometry>
@@ -21,11 +42,11 @@
 			</geometry>
 			<material name="orange"/>
-		</visual>
-	</link>
-	<xacro:servo_XM430 name="yaw" parent="base" child="connector" center_child="false" fixed_plane="back" fixed_angle="${0}"/>
+		</visual> -->
+    </link>
+	<xacro:servo_XM430 name="yaw" parent="puntilt_base" child="connector" center_child="false" fixed_plane="back" fixed_angle="${0}"/>
     <link name="connector"/>
     <xacro:servo_XM430_FR12_S102K name="pitch" parent="connector" child="hone_pitch" center_child="true" fixed_plane="bottom" fixed_angle="${pi/2}"/>
 	<link name="hone_pitch">
-		<visual>
+		<!-- <visual>
 			<origin xyz="0 0 0" rpy="0 0 0"/>
 			<geometry>
@@ -33,5 +54,5 @@
 			</geometry>
 			<material name="red"/>
-		</visual>
+		</visual> -->
 	</link>
     <xacro:sensor_d435 parent="hone_pitch" use_nominal_extrinsics="$(arg use_nominal_extrinsics)" add_plug="$(arg add_plug)" use_mesh="$(arg use_mesh)">

Commit message: small fixes

File: DynamixelPunTilt/puntilt_description/urdf/puntilt_dynamixel-2XL430_realsense-D435.urdf.xacro (robot description, xacro)
@@ -35,23 +35,8 @@
         <origin xyz="0 0 0.094" rpy="0 0 0"/>
     </joint>
-	<link name="puntilt_base">
-        <!-- <visual>
-			<origin xyz="0 0 0" rpy="0 0 0"/>
-			<geometry>
-				<box size="0.03 0.04 0.001"/>
-			</geometry>
-			<material name="orange"/>
-		</visual> -->
-    </link>
-	<xacro:servo_2XL430 name_parent="yaw" parent="puntilt_base" center_parent="false" child="pitch" center_child="true" />
-	<link name="pitch">
-		<!-- <visual>
-			<origin xyz="0 0 0" rpy="0 0 0"/>
-			<geometry>
-				<cylinder length="0.001" radius="0.01"/>
-			</geometry>
-			<material name="red"/>
-		</visual> -->
-	</link>
+	<link name="puntilt_base" />
+	<xacro:servo_2XL430 name_parent="yaw"  parent="puntilt_base" center_parent="false"
+                        name_child="pitch" child="pitch"         center_child="true" />
+	<link name="pitch" />
     <xacro:sensor_d435 parent="pitch" use_nominal_extrinsics="$(arg use_nominal_extrinsics)" add_plug="$(arg add_plug)" use_mesh="$(arg use_mesh)">
         <origin xyz="-0.01 -0.035 0.0" rpy="${-pi/2} 0 ${-pi/2}"/>

File: DynamixelPunTilt/puntilt_description/urdf/puntilt_dynamixel-XM430-double_realsense-D435.urdf.xacro (robot description, xacro)
@@ -1,6 +1,7 @@
 <?xml version="1.0"?>
-<robot name="puntilt" xmlns:xacro="http://ros.org/wiki/xacro">
-	<xacro:include filename="$(find dynamixel_description)/urdf/common_properties.xacro"/>
-	<xacro:include filename="$(find dynamixel_description)/urdf/_XM430.urdf.xacro"/>
+<robot name="puntilt"
+    xmlns:xacro="http://ros.org/wiki/xacro">
+    <xacro:include filename="$(find dynamixel_description)/urdf/common_properties.xacro"/>
+    <xacro:include filename="$(find dynamixel_description)/urdf/_XM430.urdf.xacro"/>
     <xacro:include filename="$(find realsense2_description)/urdf/_d435.urdf.xacro" />
     <!-- realsense 関連の引数 -->
@@ -10,10 +11,10 @@
     <link name="base">
         <visual>
-			<origin xyz="0 0 0" rpy="0 0 0"/>
-			<geometry>
+            <origin xyz="0 0 0" rpy="0 0 0"/>
+            <geometry>
                 <mesh filename="package://puntilt_description/meshes/waffle_base.stl" scale="0.001 0.001 0.001"/>
-			</geometry>
-			<material name="orange"/>
-		</visual>
+            </geometry>
+            <material name="orange"/>
+        </visual>
         <collision>
             <origin xyz="0 0 0.047" rpy="0 0 0"/>
@@ -25,7 +26,5 @@
             <origin xyz="${0} ${0} ${0}" rpy="${0} 0 0"/>
             <mass value="1000"/>
-            <inertia ixx="1000"  ixy="0.00" ixz="0.00"
-                                 iyy="1000" iyz="0.00"
-                                            izz="1000" />
+            <inertia ixx="1000" ixy="0.00" ixz="0.00" iyy="1000" iyz="0.00" izz="1000" />
         </inertial>
     </link>
@@ -35,5 +34,5 @@
         <origin xyz="0 0 0.094" rpy="0 0 0"/>
     </joint>
-	<link name="puntilt_base">
+    <link name="puntilt_base">
         <!-- <visual>
 			<origin xyz="0 0 0" rpy="0 0 0"/>
@@ -44,9 +43,9 @@
 		</visual> -->
     </link>
-	<xacro:servo_XM430 name="yaw" parent="puntilt_base" child="connector" center_child="false" fixed_plane="back" fixed_angle="${0}"/>
+    <xacro:servo_XM430 name="yaw" parent="puntilt_base" child="connector" center_child="false" fixed_plane="back" fixed_angle="${0}"/>
     <link name="connector"/>
     <xacro:servo_XM430_FR12_S102K name="pitch" parent="connector" child="hone_pitch" center_child="true" fixed_plane="bottom" fixed_angle="${pi/2}"/>
-	<link name="hone_pitch">
-		<!-- <visual>
+    <link name="hone_pitch">
+        <!-- <visual>
 			<origin xyz="0 0 0" rpy="0 0 0"/>
 			<geometry>
@@ -55,14 +54,14 @@
 			<material name="red"/>
 		</visual> -->
-	</link>
+    </link>
     <xacro:sensor_d435 parent="hone_pitch" use_nominal_extrinsics="$(arg use_nominal_extrinsics)" add_plug="$(arg add_plug)" use_mesh="$(arg use_mesh)">
         <origin xyz="0.035 -0.01 0.0" rpy="${-pi/2} ${0} ${0}"/>
     </xacro:sensor_d435>
-	<gazebo reference="base">
-		<material>Gazebo/Orange</material>
-	</gazebo>
-	<gazebo reference="hone">
-		<material>Gazebo/Red</material>
-	</gazebo>
+    <gazebo reference="base">
+        <material>Gazebo/Orange</material>
+    </gazebo>
+    <gazebo reference="hone">
+        <material>Gazebo/Red</material>
+    </gazebo>
     <!--ros_controlプラグインをロード-->
     <gazebo>
